File: sgd_10x15/GlassIDC_Mounted_10x15mm.kicad_pcb (KiCad board)
At the start: 4 copper layers, 36.8 x 36.8 mm, 0 parts

Commit message: finished design and gerbs
Parts:
- added REF**: MountingHole_2.5mm_Pad, MountingHole:MountingHole_2.5mm_Pad, F.Cu at (137.0, 93.5)
- added REF**: MountingHole_2.5mm_Pad, MountingHole:MountingHole_2.5mm_Pad, F.Cu at (159.9, 116.3)
- added REF**: MountingHole_2.5mm_Pad, MountingHole:MountingHole_2.5mm_Pad, F.Cu at (137.1, 116.3)
- added REF**: MountingHole_2.5mm_Pad, MountingHole:MountingHole_2.5mm_Pad, F.Cu at (159.9, 93.5)
Routing:
- net (no net): track 53.6 -> 308.7 mm, vias 74 -> 73
- added copper zone on B.Cu, net (none)
Other:
- copper layers 4 -> 2

Commit message: pcb v3
Routing:
- net (no net): vias 73 -> 77
